File: VCU.kicad_pcb (KiCad board)
At the start: 2 copper layers, 44.3 x 40.3 mm, 38 parts, among them J1 Conn_02x03_Top_Bottom, J2 2x3_Conn, J3 USB_C_Receptacle_USB2.0_14P, J4 Conn_01x02, SW1 SW_Push, SW2 SW_Push, U1 ESP32-S3-WROOM-1, U2 LM1117DT-3.3, U3 SN65HVD230, U4 USBLC6-2SC6, U6 MCP6001-OT

Commit message: Add silkscreen Labels, Add gnd pin to CANTrans
Connections:
- C1 pad 2: Net-(U3-GND) -> GND
- U3 pad 2: Net-(U3-GND) -> GND
Routing:
- net Net-(U3-GND): track 2.41 -> 0.00 mm
- net GND: track 8.83 -> 11.2 mm, vias 85 -> 86
Other:
- board text added: "12V"
- board text added: "CANH"
- board text added: "CANL"
- board text added: "GND"
- board text added: "IO1"
- board text added: "IO2"
- board text added: "IO5"
- board text added: "IO6"
