File: VCU.kicad_pcb (KiCad board)
At the start: 2 copper layers, 44.3 x 40.3 mm, 36 parts, among them J2 2x3_Conn, J3 USB_C_Receptacle_USB2.0_14P, U1 ESP32-S3-WROOM-1, U2 LM1117DT-3.3, U3 SN65HVD230, U4 USBLC6-2SC6, U6 MCP6001-OT

Commit message: Do Layout
Yuh
Parts:
- added C12: 100 nF, Capacitor_SMD:C_0805_2012Metric, F.Cu at (72.4, 69.5)
- added C13: 100 nF, Capacitor_SMD:C_0805_2012Metric, F.Cu at (73.6, 78.4)
- added C14: 100 nF, Capacitor_SMD:C_0805_2012Metric, B.Cu at (82.0, 78.5)
- added C15: 27pF, Capacitor_SMD:C_0805_2012Metric, F.Cu at (69.6, 74.2)
- added C16: 27pF, Capacitor_SMD:C_0805_2012Metric, F.Cu at (69.6, 76.2)
- added J1: Conn_02x03_Top_Bottom, Connector_PinHeader_2.54mm:PinHeader_2x03_P2.54mm_Vertical, F.Cu at (110.0, 49.5)
- added J5: Conn_01x02, Connector_Molex:Molex_Mini-Fit_Jr_5566-02A_2x01_P4.20mm_Vertical, F.Cu at (109.2, 79.0)
- added R16: 60, Resistor_SMD:R_0805_2012Metric, F.Cu at (80.1, 79.5)
- added R26: 10k, Resistor_SMD:R_0805_2012Metric, B.Cu at (96.1, 61.5)
- added R27: 10k, Resistor_SMD:R_0805_2012Metric, B.Cu at (84.5, 56.2)
- added R28: 60, Resistor_SMD:R_0805_2012Metric, F.Cu at (80.1, 77.5)
- added U5: MCP2518FD-xQBB, Package_DFN_QFN:DFN-14-1EP_3x4.5mm_P0.65mm_EP1.65x4.25mm, B.Cu at (71.0, 70.1)
- added U7: PTCAN3413DR, KiCADv6:SOIC8_D_TEX, B.Cu at (76.3, 78.4)
- added Y1: 40Mhz Crystal, Crystal:Crystal_SMD_3225-4Pin_3.2x2.5mm, B.Cu at (69.5, 75.0)
- U4: footprint SK's_Components:ESD_SOT-23-6 -> Package_TO_SOT_SMD:SOT-23-6
Connections:
- net Vin(12V) renamed Vin(5V)
- C1 pad 2: Net-(U3-GND) -> GND
- C2 pad 1: Net-(U3-Vref) -> +3.3V
- J2 pad 3: CAN- -> /CANFD-
- J2 pad 6: CAN+ -> /CANFD+
- J3 pad S1: GND -> (no net)
- R15 pad 1: GPIO_TEST1 -> Net-(U6--)
- R15 pad 2: Net-(U6--) -> GPIO_TEST1
- U1 pad 10: unconnected-(U1-IO17-Pad10) -> /INT
- U1 pad 19: unconnected-(U1-IO11-Pad19) -> /MOSI
- U1 pad 20: unconnected-(U1-IO12-Pad20) -> /SPIClk
- U1 pad 21: unconnected-(U1-IO13-Pad21) -> /MISO
- U1 pad 22: unconnected-(U1-IO14-Pad22) -> /CS
- U1 pad 32: unconnected-(U1-IO39-Pad32) -> /IO1
- U1 pad 33: unconnected-(U1-IO40-Pad33) -> /IO2
- U1 pad 34: unconnected-(U1-IO41-Pad34) -> /IO3
- U1 pad 35: unconnected-(U1-IO42-Pad35) -> /IO4
- U1 pad 38: unconnected-(U1-IO2-Pad38) -> /IO5
- U1 pad 39: unconnected-(U1-IO1-Pad39) -> /IO6
- U3 pad 2: Net-(U3-GND) -> GND
- U3 pad 5: Net-(U3-Vref) -> +3.3V
Routing:
- net /CANFD+: track 0.00 -> 41.1 mm, vias 0 -> 1
- net /CANFD-: track 0.00 -> 41.1 mm, vias 0 -> 1
- net /INT: track 0.00 -> 30.8 mm, vias 0 -> 3
- net /SPIClk: track 0.00 -> 30.6 mm, vias 0 -> 1
- net /MOSI: track 0.00 -> 28.1 mm, vias 0 -> 1
- net /CS: track 0.00 -> 27.4 mm, vias 0 -> 1
- net /MISO: track 0.00 -> 27.2 mm, vias 0 -> 1
- net /IO3: track 0.00 -> 10.7 mm, vias 0 -> 1
- net /TX: track 0.00 -> 10.3 mm, vias 0 -> 2
- net /IO1: track 0.00 -> 9.83 mm, vias 0 -> 1
- net /IO5: track 0.00 -> 8.78 mm
- net +3.3V: track 72.6 -> 80.7 mm, vias 8 -> 12
- net /IO4: track 0.00 -> 7.73 mm, vias 0 -> 1
- net /IO2: track 0.00 -> 7.17 mm, vias 0 -> 1
- net /IO6: track 0.00 -> 5.71 mm
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Other:
- board size 44.3 x 40.3 mm -> 45.6 x 40.3 mm
- board text added: "CanH"
- board text added: "CanL"
- board text added: "GND"
- board text added: "GPIO1"
- board text added: "GPIO2"
- board text added: "IO1"
- board text added: "IO6"
- board text added: "Vin"

Commit message: ERC, DRC
Parts:
- removed BOOTLOAD: SW_Push, SK's_Components:Button_MJTP1250
- removed Enable Switch: SW_Push, SK's_Components:Button_MJTP1250
- added SW2: SW_Push, SK's_Components:Button_MJTP1250, F.Cu at (75.5, 45.8)
- added SW3: SW_Push, SK's_Components:Button_MJTP1250, F.Cu at (102.5, 66.1)
Connections:
- R15 pad 1: Net-(U6--) -> GPIO_TEST1
- R15 pad 2: GPIO_TEST1 -> Net-(U6--)
Routing:
- net +3.3V: track 80.7 -> 99.1 mm, vias 12 -> 17
- net CAN-: track 21.0 -> 18.8 mm
- net CAN+: track 19.9 -> 18.8 mm
- net /CS: track 27.4 -> 28.3 mm, vias 1 -> 3
- net Net-(U5-OSC1): track 3.09 -> 3.65 mm

Commit message: fix SS
Parts:
- SW2: value SW_Push -> ENABLE
- renumbered SW3 to BOOT
Changed lines of the file:
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@@
 			)
 		)
-		(property "Value" "SW_Push"
+		(property "Value" "ENABLE"
 			(at 3.25 2.8 90)
 			(layer "F.SilkS")
@@
 		(descr "tactile push button, 6x3.5mm, https://www.apem.com/idec-apem/en_US/PCB-switches/Tactile-Switches/MJTP-6mm-through-hole/c/MJTP_6mm_through%20hole?page=1")
 		(tags "PHAP3362A 6mm tact sw THT")
-		(property "Reference" "SW3"
-			(at 3.42 -2.7 90)
+		(property "Reference" "BOOT"
+			(at 2.895 2.475 90)
 			(layer "F.SilkS")
 			(effects
@@
 		(net "+3.3V")
 	)
-	(segment
-		(start 101.325 66)
-		(end 102.5 66)
-		(width 0.3)
-		(layer "F.Cu")
-		(net "BOOTLOAD")
-	)
-	(segment
-		(start 103 66)
-		(end 104 65)
-		(width 0.3)
-		(layer "F.Cu")
-		(net "BOOTLOAD")
-	)
-	(segment
-		(start 102.5 66)
-		(end 103 66)
-		(width 0.3)
-		(layer "F.Cu")
-		(net "BOOTLOAD")
-	)
-	(segment
-		(start 104 65)
-		(end 104 62.31)
-		(width 0.3)
-		(layer "F.Cu")
-		(net "BOOTLOAD")
-	)
-	(segment
-		(start 98.825 63.5)
-		(end 101.325 66)
-		(width 0.3)
-		(layer "F.Cu")
-		(net "BOOTLOAD")
-	)
-	(segment
-		(start 104 62.31)
-		(end 102 60.31)
-		(width 0.3)
-		(layer "F.Cu")
-		(net "BOOTLOAD")
-	)
 	(via
 		(at 68.4 74.15)
@@
 		(net "/CS")
 	)
+	(segment
+		(start 101.325 66)
+		(end 102.5 66)
+		(width 0.3)
+		(layer "F.Cu")
+		(net "BOOTLOAD")
+	)
+	(segment
+		(start 103 66)
+		(end 104 65)
+		(width 0.3)
+		(layer "F.Cu")
+		(net "BOOTLOAD")
+	)
+	(segment
+		(start 102.5 66)
+		(end 103 66)
+		(width 0.3)
+		(layer "F.Cu")
+		(net "BOOTLOAD")
+	)
+	(segment
+		(start 104 65)
+		(end 104 62.31)
+		(width 0.3)
+		(layer "F.Cu")
+		(net "BOOTLOAD")
+	)
+	(segment
+		(start 98.825 63.5)
+		(end 101.325 66)
+		(width 0.3)
+		(layer "F.Cu")
+		(net "BOOTLOAD")
+	)
+	(segment
+		(start 104 62.31)
+		(end 102 60.31)
+		(width 0.3)
+		(layer "F.Cu")
+		(net "BOOTLOAD")
+	)
 	(via
 		(at 102 53.96)
@@
 		(net "Vin(5V)")
 	)
+	(segment
+		(start 105.435 68.225)
+		(end 105.435 66.675)
+		(width 0.3)
+		(layer "F.Cu")
+		(net "Net-(C5-Pad1)")
+	)
+	(segment
+		(start 105.435 66.675)
+		(end 105.885 66.225)
+		(width 0.3)
+		(layer "F.Cu")
+		(net "Net-(C5-Pad1)")
+	)
+	(segment
+		(start 107.885 66.225)
+		(end 105.885 66.225)
+		(width 0.3)
+		(layer "F.Cu")
+		(net "Net-(C5-Pad1)")
+	)
 	(via
 		(at 105.885 64.4)
@@
 		(net "Net-(U5-OSC2)")
 	)
+	(via
+		(at 81 78)
+		(size 0.6)
+		(drill 0.3)
+		(layers "F.Cu" "B.Cu")
+		(net "Net-(C14-Pad1)")
+	)
+	(via
+		(at 81 79)
+		(size 0.6)
+		(drill 0.3)
+		(layers "F.Cu" "B.Cu")
+		(net "Net-(C14-Pad1)")
+	)
 	(segment
 		(start 74.5525 62.2)
@@
 		(net "/RX")
 	)
-	(segment
-		(start 105.435 68.225)
-		(end 105.435 66.675)
-		(width 0.3)
-		(layer "F.Cu")
-		(net "Net-(C5-Pad1)")
-	)
-	(segment
-		(start 105.435 66.675)
-		(end 105.885 66.225)
-		(width 0.3)
-		(layer "F.Cu")
-		(net "Net-(C5-Pad1)")
-	)
-	(segment
-		(start 107.885 66.225)
-		(end 105.885 66.225)
-		(width 0.3)
-		(layer "F.Cu")
-		(net "Net-(C5-Pad1)")
-	)
-	(via
-		(at 81 78)
-		(size 0.6)
-		(drill 0.3)
-		(layers "F.Cu" "B.Cu")
-		(net "Net-(C14-Pad1)")
-	)
-	(via
-		(at 81 79)
-		(size 0.6)
-		(drill 0.3)
-		(layers "F.Cu" "B.Cu")
-		(net "Net-(C14-Pad1)")
-	)
 	(zone

Commit message: Fix weirdly appearing DRC Issues
Parts:
- removed U2: LM1117DT-3.3, Package_TO_SOT_SMD:TO-252-3_TabPin2
- added U8: AP2112K-3.3, Package_TO_SOT_SMD:SOT-23-5, F.Cu at (79.0, 72.0)
- C7: moved to B.Cu
- SW2: value ENABLE -> SW_Push
- moved C7 2.93 mm to (81.0, 72.0), turned to 0 degrees
Connections:
- C2 pad 1: +3.3V -> Net-(U3-Vref)
- U1 pad 16: unconnected-(U1-IO46-Pad16) -> /IO6
- U1 pad 26: unconnected-(U1-IO45-Pad26) -> /IO5
- U1 pad 36: CAN_RX -> unconnected-(U1-RXD0-Pad36)
- U1 pad 37: CAN_TX -> unconnected-(U1-TXD0-Pad37)
- U1 pad 38: /IO5 -> CAN_RX
- U1 pad 39: /IO6 -> CAN_TX
- U3 pad 5: +3.3V -> Net-(U3-Vref)
Routing:
- net /IO6: track 5.71 -> 34.0 mm, vias 0 -> 1
- net /IO5: track 8.78 -> 24.1 mm, vias 0 -> 1
- net Vin(5V): track 7.95 -> 14.5 mm, vias 0 -> 1
- net +3.3V: track 99.1 -> 93.5 mm, vias 17 -> 15
- net Net-(U3-Vref): track 0.00 -> 3.27 mm, vias 0 -> 2
- net CAN_TX: track 7.63 -> 10.1 mm
- net CAN_RX: track 5.65 -> 8.14 mm
- net GND: vias 80 -> 114

Commit message: Add bom
Parts:
- removed J3: USB_C_Receptacle_USB2.0_14P, SK's_Components:USB_C_HRO_TYPE-C-31-M-14
- removed R29, R8, R9: 60, Resistor_SMD:R_0805_2012Metric
- added C17: 100 nF, Capacitor_SMD:C_0805_2012Metric, F.Cu at (75.8, 73.4)
- added J4: UJ20-C-H-G-SMT-4-P16-TR, UJ20-C-H-G-SMT-4-P16-TR:SAMESKY_UJ20-C-H-G-SMT-4-P16-TR, F.Cu at (67.1, 59.8)
- moved R7 0.11 mm to (77.2, 62.1)
- moved R6 0.10 mm to (76.3, 56.8)
Connections:
- U3 pad 1: Net-(U3-D) -> CAN_TX
- U3 pad 4: Net-(U3-R) -> CAN_RX
- U3 pad 8: Net-(U3-Rs) -> GND
Routing:
- net Net-(U3-Rs): track 9.73 -> 0.00 mm, vias 2 -> 0
- net USB_D-: track 8.56 -> 14.6 mm
- net CAN_TX: track 10.1 -> 15.9 mm
- net Net-(U3-D): track 4.68 -> 0.00 mm
- net CAN_RX: track 8.14 -> 12.5 mm
- net GND: track 11.2 -> 8.14 mm, vias 114 -> 115
- net USB_D+: track 8.47 -> 11.4 mm, vias 0 -> 2
- net +3.3V: track 93.5 -> 96.2 mm
- net Net-(U3-R): track 2.49 -> 0.00 mm
- net VBUS: track 11.8 -> 12.3 mm

Commit message: lol
Routing:
- net Vin(5V): track 14.5 -> 12.5 mm
Changed lines of the file:
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@@
 	)
 	(segment
-		(start 81.315 73.685)
-		(end 80.63 73)
+		(start 81.9 72.6)
+		(end 81.9 72)
 		(width 1)
 		(layer "F.Cu")
@@
 	)
 	(segment
-		(start 83.7 74.1)
-		(end 81.73 74.1)
-		(width 1)
-		(layer "F.Cu")
-		(net "Vin(5V)")
-	)
-	(segment
-		(start 86.75 74.1)
-		(end 83.7 74.1)
+		(start 81.9 72)
+		(end 83.3 72)
 		(width 1)
 		(layer "F.Cu")
@@
 	)
 	(segment
-		(start 81.315 73.685)
-		(end 81.9 73.1)
+		(start 83.3 72)
+		(end 83.8 72.5)
 		(width 1)
 		(layer "F.Cu")
@@
 	)
 	(segment
-		(start 81.9 73.1)
-		(end 81.9 72)
+		(start 81.5 73)
+		(end 81.9 72.6)
 		(width 1)
 		(layer "F.Cu")
@@
 	)
 	(segment
-		(start 80.63 73)
-		(end 80.1375 73)
+		(start 83.8 72.5)
+		(end 88.35 72.5)
 		(width 1)
 		(layer "F.Cu")
@@
 	)
 	(segment
-		(start 81.73 74.1)
-		(end 81.315 73.685)
+		(start 80.1375 73)
+		(end 81.5 73)
 		(width 1)
 		(layer "F.Cu")
-		(net "Vin(5V)")
-	)
-	(segment
-		(start 88.35 72.5)
-		(end 86.75 74.1)
-		(width 1)
-		(layer "F.Cu")

Commit message: add gerbs
Parts:
- added G***: LOGO, LOGO, B.Cu at (93.3, 52.9)
- SW2: value SW_Push -> ENABLE
