File: _autosave-VCU.kicad_pcb (KiCad board)
At the start: 2 copper layers, 45.6 x 40.3 mm, 49 parts, among them J1 Conn_02x03_Top_Bottom, J2 2x3_Conn, J4 UJ20-C-H-G-SMT-4-P16-TR, J5 Conn_01x02, SW2 ENABLE, U1 ESP32-S3-WROOM-1, U3 SN65HVD230, U4 USBLC6-2SC6, U5 MCP2518FD-xQBB, U6 MCP6001-OT, U7 PTCAN3413DR, U8 AP2112K-3.3, Y1 40Mhz Crystal

Commit message: Fix Gerbs
Parts:
- moved G*** 1.40 mm to (93.3, 54.3)
Changed lines of the file:
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@@
 	(footprint "LOGO"
 		(layer "B.Cu")
-		(at 93.3 52.9 180)
+		(at 93.3 54.3 180)
 		(property "Reference" "G***"
 			(at 0 0 0)
@@
 	(dimension
 		(type orthogonal)
-		(layer "F.Fab")
+		(layer "F.Cu")
 		(pts
-			(xy 66.9 82.2) (xy 111.2 82.2)
-		)
-		(height 7.2)
+			(xy 112.5 82.2) (xy 66.9 82.2)
+		)
+		(height 8.9)
 		(orientation 0)
 		(format
@@
 			(keep_text_aligned yes)
 		)
-		(gr_text "44.3"
-			(at 89.05 87.6 0)
-			(layer "F.Fab")
-			(effects
-				(font
+		(gr_text "45.6"
+			(at 89.7 89.3 0)
+			(layer "F.Cu")
+			(effects
+				(font
